File: Hardware/ADF4351_synthesizer/UART_USB_Interface.kicad_sch (KiCad schematic)
At the start: 21 parts, among them J3 USB_C_Receptacle_USB2.0_16P, U1 FT231XQ, U6 AZ1117ID-3.3TRG1

Commit message: Updating schematic
Parts:
- removed C23, C24, C25: 10uF, Capacitor_Tantalum_SMD:CP_EIA-3216-18_Kemet-A, symbol Device:C_Polarized_Small_US
- removed U6: AZ1117ID-3.3TRG1, Package_TO_SOT_SMD:TO-252-2, symbol Regulator_Linear:AZ1117-3.3
Other:
- note removed: "1 Amp Max"
- note removed: "ADM7154"
- note removed: "ADM7154ARDZ-3.3-R7"
- note removed: "Not Recommended for new designs"

Commit message: Starting to organize PCB Layout
Parts:
- renumbered C17 to C41, C18 to C42, C19 to C43, C20 to C44, C21 to C45, C22 to C46, D6 to D4, D8 to D5, D9 to D6, J3 to J6, L2 to L5, R12 to R15, R13 to R16, R14 to R17, R15 to R18, R16 to R19, U1 to U5
