File: Hardware/ADF4351_synthesizer/ADF4351_synthesizer.kicad_sch (KiCad schematic)
At the start: 21 parts, among them J1 AVR-UPDI-6, J2 Conn_01x04_Socket, J4 Conn_02x03_Odd_Even, SW1 SW_Push, U2 AVR128DA32x-xPT

Commit message: Updating schematic
Parts:
- removed J2: Conn_01x04_Socket, symbol Connector:Conn_01x04_Socket
- removed J4: Conn_02x03_Odd_Even, symbol Connector_Generic:Conn_02x03_Odd_Even
- added J4: Conn_01x05_Socket, symbol Connector:Conn_01x05_Socket
- added R8, R9: 5.1k, Resistor_SMD:R_0603_1608Metric, symbol Device:R_Small_US
- added U3: AT24CS16-STUM, Package_SO:SOIC-8_3.9x4.9mm_P1.27mm, symbol Memory_EEPROM:AT24CS16-STUM
Connections:
- net +3V3: now also R8.1, R9.1, U3.4 (VCC)
- net GND: now also J4.5 (Pin_5), U3.2 (GND), U3.5 (WP)
- net MISO: now also J4.1 (Pin_1)
- net MOSI: now also J4.2 (Pin_2)
- net SCLK: now also J4.4 (Pin_4)
- net ~{SYNTH_CS}: now also J4.3 (Pin_3)
- net SCL: now reaches U2.1 (PA3)
- net SCL: now also R9.2, U3.1 (SCL)
- net SDA: now reaches U2.32 (PA2)
- net SDA: now also R8.2, U3.3 (SDA)
- net XO_EN: now reaches U2.8 (PC2)
Other:
- moved on the sheet: J1

Commit message: Starting to organize PCB Layout
Parts:
- removed R4, R5, R6, R7: 27, Resistor_SMD:R_0603_1608Metric, symbol Device:R_Small_US
- removed U3: AT24CS16-STUM, Package_SO:SOIC-8_3.9x4.9mm_P1.27mm, symbol Memory_EEPROM:AT24CS16-STUM
- added U6: AT24CS16-STUM, Package_TO_SOT_SMD:SOT-23-5, symbol Memory_EEPROM:AT24CS16-STUM
- J2: renamed from J4; footprint (none) -> Connector_PinHeader_1.27mm:PinHeader_1x05_P1.27mm_Vertical
- renumbered C4 to C1, C7 to C2, C9 to C3, C5 to C4, C8 to C5, C10 to C7, R3 to R1, R8 to R2, R9 to R3, R1 to R4, R2 to R5, U2 to U1
Connections:
- net +3V3: now also U6.4 (VCC)
- net GND: now also U6.2 (GND), U6.5 (WP)
- net MISO: now also J2.3 (Pin_3), U1.3 (PA5); no longer J2.1 (Pin_1)
- net MOSI: now also J2.4 (Pin_4), U1.2 (PA4); no longer J2.2 (Pin_2)
- net SCL: now also U6.1 (SCL)
- net SCLK: now also J2.2 (Pin_2), U1.4 (PA6); no longer J2.4 (Pin_4)
- net SDA: now also U6.3 (SDA)
- net ~{SYNTH_CS}: now also J2.1 (Pin_1), U1.5 (PA7); no longer J2.3 (Pin_3)
Other:
- note added: "SPI Header"
- company: (none) -> openEPR
- title: (none) -> ADF4351 Synthesizer

Commit message: Updating board
Parts:
- removed C2: 100nF, Capacitor_SMD:C_0402_1005Metric, symbol Device:C_Small
- removed C5: 10nF, Capacitor_SMD:C_0402_1005Metric, symbol Device:C_Small
Changed lines of the file:
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@@
 	)
 	(junction
-		(at 82.55 24.13)
-		(diameter 0)
-		(color 0 0 0 0)
-	)
-	(junction
 		(at 44.45 67.31)
 		(diameter 0)
@@
 	)
 	(junction
-		(at 100.33 29.21)
-		(diameter 0)
-		(color 0 0 0 0)
-	)
-	(junction
-		(at 69.85 29.21)
-		(diameter 0)
-		(color 0 0 0 0)
-	)
-	(junction
-		(at 83.82 24.13)
+		(at 83.82 26.67)
 		(diameter 0)
 		(color 0 0 0 0)
@@
 	)
 	(junction
-		(at 85.09 24.13)
-		(diameter 0)
-		(color 0 0 0 0)
-	)
-	(junction
 		(at 85.09 29.21)
 		(diameter 0)
@@
 	(wire
 		(pts
-			(xy 90.17 24.13) (xy 85.09 24.13)
-		)
-		(stroke
-			(width 0)
-			(type default)
-		)
-	)
-	(wire
-		(pts
 			(xy 44.45 67.31) (xy 40.64 67.31)
 		)
@@
 	(wire
 		(pts
-			(xy 82.55 29.21) (xy 82.55 34.29)
-		)
-		(stroke
-			(width 0)
-			(type default)
-		)
-	)
-	(wire
-		(pts
 			(xy 144.78 34.29) (xy 147.32 34.29)
 		)
@@
 	(wire
 		(pts
-			(xy 82.55 24.13) (xy 82.55 29.21)
+			(xy 82.55 26.67) (xy 82.55 29.21)
 		)
 		(stroke
@@
 	(wire
 		(pts
-			(xy 95.25 24.13) (xy 100.33 24.13)
-		)
-		(stroke
-			(width 0)
-			(type default)
-		)
-	)
-	(wire
-		(pts
 			(xy 105.41 161.29) (xy 105.41 160.02)
 		)
@@
 	(wire
 		(pts
-			(xy 83.82 21.59) (xy 83.82 24.13)
+			(xy 83.82 24.13) (xy 83.82 26.67)
 		)
 		(stroke
@@
 	(wire
 		(pts
-			(xy 80.01 24.13) (xy 82.55 24.13)
-		)
-		(stroke
-			(width 0)
-			(type default)
-		)
-	)
-	(wire
-		(pts
-			(xy 69.85 24.13) (xy 74.93 24.13)
-		)
-		(stroke
-			(width 0)
-			(type default)
-		)
-	)
-	(wire
-		(pts
-			(xy 100.33 24.13) (xy 100.33 29.21)
-		)
-		(stroke
-			(width 0)
-			(type default)
-		)
-	)
-	(wire
-		(pts
 			(xy 146.05 24.13) (xy 147.32 24.13)
 		)
@@
 	(wire
 		(pts
-			(xy 85.09 29.21) (xy 85.09 34.29)
-		)
-		(stroke
-			(width 0)
-			(type default)
-		)
-	)
-	(wire
-		(pts
 			(xy 105.41 69.85) (xy 107.95 69.85)
 		)
@@
 	(wire
 		(pts
-			(xy 69.85 24.13) (xy 69.85 29.21)
-		)
-		(stroke
-			(width 0)
-			(type default)
-		)
-	)
-	(wire
-		(pts
 			(xy 115.57 154.94) (xy 116.84 154.94)
 		)
@@
 	(wire
 		(pts
-			(xy 83.82 24.13) (xy 82.55 24.13)
+			(xy 83.82 26.67) (xy 82.55 26.67)
 		)
 		(stroke
@@
 	(wire
 		(pts
-			(xy 85.09 24.13) (xy 85.09 29.21)
+			(xy 82.55 29.21) (xy 82.55 34.29)
 		)
 		(stroke
@@
 	(wire
 		(pts
-			(xy 85.09 24.13) (xy 83.82 24.13)
+			(xy 85.09 26.67) (xy 85.09 29.21)
+		)
+		(stroke
+			(width 0)
+			(type default)
+		)
+	)
+	(wire
+		(pts
+			(xy 85.09 26.67) (xy 83.82 26.67)
 		)
 		(stroke
@@
 		)
 	)
+	(wire
+		(pts
+			(xy 85.09 29.21) (xy 85.09 34.29)
+		)
+		(stroke
+			(width 0)
+			(type default)
+		)
+	)
 	(text "SPI Header"
 		(exclude_from_sim no)
@@
 	)
 	(symbol
-		(lib_id "Device:C_Small")
-		(at 92.71 24.13 90)
-		(unit 1)
-		(exclude_from_sim no)
-		(in_bom yes)
-		(on_board yes)
-		(dnp no)
-		(property "Reference" "C5"
-			(at 96.266 23.114 90)
-			(effects
-				(font
-					(size 1.27 1.27)
-				)
-			)
-		)
-		(property "Value" "10nF"
-			(at 89.154 22.86 90)
-			(effects
-				(font
-					(size 1.27 1.27)
-				)
-			)
-		)
-		(property "Footprint" "Capacitor_SMD:C_0402_1005Metric"
-			(at 92.71 24.13 0)
-			(effects
-				(font
-					(size 1.27 1.27)
-				)
-				(hide yes)
-			)
-		)
-		(property "Datasheet" "~"
-			(at 92.71 24.13 0)
-			(effects
-				(font
-					(size 1.27 1.27)
-				)
-				(hide yes)
-			)
-		)
-		(property "Description" "Unpolarized capacitor, small symbol"
-			(at 92.71 24.13 0)
-			(effects
-				(font
-					(size 1.27 1.27)
-				)
-				(hide yes)
-			)
-		)
-		(pin "2"
-		)
-		(pin "1"
-		)
-		(instances
-			(project "ADF4351_synthesizer"
-				(path "/803fce22-1ef3-4294-841a-dc90f5d59ce1"
-					(reference "C5")
-					(unit 1)
-				)
-			)
-		)
-	)
-	(symbol
 		(lib_id "power:GND")
 		(at 85.09 101.6 0)
@@
 	(symbol
 		(lib_id "power:+3V3")
-		(at 83.82 21.59 0)
+		(at 83.82 24.13 0)
 		(unit 1)
 		(exclude_from_sim no)
@@
 		(dnp no)
 		(property "Reference" "#PWR05"
-			(at 83.82 25.4 0)
+			(at 83.82 27.94 0)
 			(effects
 				(font
@@
 		)
 		(property "Value" "+3V3"
-			(at 83.82 18.288 0)
+			(at 83.82 20.828 0)
 			(effects
 				(font
@@
 		)
 		(property "Footprint" ""
-			(at 83.82 21.59 0)
+			(at 83.82 24.13 0)
 			(effects
 				(font
@@
 		)
 		(property "Datasheet" ""
-			(at 83.82 21.59 0)
+			(at 83.82 24.13 0)
 			(effects
 				(font
@@
 		)
 		(property "Description" "Power symbol creates a global label with name \"+3V3\""
-			(at 83.82 21.59 0)
+			(at 83.82 24.13 0)
 			(effects
 				(font
@@
 					(unit 1)
 				)
-			)
-		)
-	)
-	(symbol
-		(lib_id "Device:C_Small")
-		(at 77.47 24.13 90)
-		(unit 1)
-		(exclude_from_sim no)
-		(in_bom yes)
-		(on_board yes)
-		(dnp no)
-		(property "Reference" "C2"
-			(at 80.264 22.86 90)
-			(effects
-				(font
-					(size 1.27 1.27)
-				)
-			)
-		)
-		(property "Value" "100nF"
-			(at 73.406 22.606 90)
-			(effects
-				(font
-					(size 1.27 1.27)
-				)
-			)
-		)
-		(property "Footprint" "Capacitor_SMD:C_0402_1005Metric"
-			(at 77.47 24.13 0)
-			(effects
-				(font
-					(size 1.27 1.27)
-				)
-				(hide yes)
-			)
-		)
-		(property "Datasheet" "~"
-			(at 77.47 24.13 0)
-			(effects
-				(font
-					(size 1.27 1.27)
-				)
-				(hide yes)
-			)
-		)
-		(property "Description" "Unpolarized capacitor, small symbol"
-			(at 77.47 24.13 0)
-			(effects
-				(font
-					(size 1.27 1.27)
-				)
-				(hide yes)
-			)
-		)
-		(pin "2"
-		)
-		(pin "1"
-		)
-		(instances
-			(project "ADF4351_synthesizer"
-				(path "/803fce22-1ef3-4294-841a-dc90f5d59ce1"
-					(reference "C2")
-					(unit 1)
-				)
