File: Hardware/ADF4351_synthesizer/ADF4351_synthesizer.kicad_pcb (KiCad board)
At the start: 4 copper layers, 89 parts, among them J1 AVR-UPDI-6, J2 Conn_01x05_Socket, J3 SMA-J-P-H-ST-EM1, J4 SMA-J-P-H-ST-EM1, J5 SMA-J-P-H-ST-EM1, J6 USB_C_Receptacle_USB2.0_16P, SW1 SW_Push, U1 AVR128DA32x-xPT, U3 ADM7150ARDZ-3.3-R7, U4 ADF4351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

Commit message: Updating board
Parts:
- removed C5: 10nF, Capacitor_SMD:C_0402_1005Metric
- moved C25 95.4 mm to (176.1, 98.4), turned to 90 degrees
- moved C23 93.9 mm to (176.1, 102.4), turned to -90 degrees
- moved C21 93.6 mm to (170.2, 105.2), turned to -90 degrees
- moved C26 93.3 mm to (175.1, 98.4), turned to 90 degrees
- moved C22 92.7 mm to (171.2, 104.6), turned to -90 degrees
- moved C24 91.9 mm to (175.1, 102.4), turned to -90 degrees
- moved C32 90.7 mm to (168.0, 103.0), turned to 90 degrees
- moved C27 89.7 mm to (174.0, 96.0), turned to 180 degrees
- moved C28 89.1 mm to (174.0, 97.0), turned to 180 degrees
- moved C31 83.7 mm to (167.0, 103.0), turned to 90 degrees
- moved C34 75.3 mm to (166.1, 86.4), turned to 180 degrees
- moved C33 75.1 mm to (162.4, 89.9)
- moved R10 72.0 mm to (166.2, 91.7), turned to 180 degrees
- moved C35 70.9 mm to (162.4, 86.2), turned to 180 degrees
- moved R11 70.6 mm to (166.2, 88.1), turned to 180 degrees
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Connections:
- C2 pad 1: GND -> +3.3VA
- C2 pad 2: +3V3 -> GND

Commit message: Working on Board Layout
Parts:
- moved C12 91.6 mm to (173.0, 94.9), turned to 180 degrees
- moved C14 91.0 mm to (173.0, 95.9), turned to 180 degrees
- moved C18 90.1 mm to (168.4, 96.0)
- moved C19 89.5 mm to (168.4, 97.0)
- moved C16 87.8 mm to (170.3, 96.0)
- moved C17 87.3 mm to (170.3, 97.0), turned to 180 degrees
- moved C29 84.3 mm to (167.5, 99.3)
- moved C30 83.7 mm to (167.5, 100.3)
- moved R9 78.0 mm to (170.1, 94.6), turned to 180 degrees
- moved R2 51.6 mm to (80.1, 72.5)
- moved R3 51.6 mm to (80.1, 75.1)
- moved C21 2.68 mm to (172.8, 105.4), turned to 0 degrees
- moved C22 1.67 mm to (172.8, 104.4), turned to 0 degrees
- moved C28 0.90 mm to (174.9, 96.9)
- moved C27 0.90 mm to (174.9, 95.9)
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